File: Hackboard.kicad_pcb (KiCad board)
At the start: 4 copper layers, 110.2 x 53.8 mm, 67 parts, among them J1 Conn_01x31_Socket, J2 Micro_SD_Card, J3 Conn_01x31_Socket, J5 Conn_02x02_Counter_Clockwise, J6 USB_C_Receptacle_USB2.0_16P, J7 Barrel_Jack_Switch, Q1 NMOS, Q2 NMOS, Q3 NMOS, SW1 SW_DPST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

Commit message: Finish PCB
Parts:
- added G***: LOGO, Symbol:logo, F.Cu at (156.7, 84.3)
- added R17: 50k, Resistor_SMD:R_0603_1608Metric, F.Cu at (180.3, 97.5)
- added R18: 50k, Resistor_SMD:R_0603_1608Metric, F.Cu at (178.1, 93.3)
- added R19: 50k, Resistor_SMD:R_0603_1608Metric, F.Cu at (179.8, 93.3)
- added R20: 50k, Resistor_SMD:R_0603_1608Metric, F.Cu at (180.8, 89.7)
- added REF**: OSHW-Logo2_7.3x6mm_SilkScreen, Symbol:OSHW-Logo2_7.3x6mm_SilkScreen, B.Cu at (155.4, 86.4)
- added REF**: KiCad-Logo2_5mm_SilkScreen, Symbol:KiCad-Logo2_5mm_SilkScreen, B.Cu at (166.4, 85.9)
- SW1: value SW_DPST -> SW_SPST
- moved JP2 13.6 mm to (189.0, 107.2)
Connections:
- JP2 pad 1: PWM_PIN2 -> Net-(JP2-A)
- JP2 pad 2: Net-(JP2-B) -> PWM_PIN2_O
- U6 pad 14: Net-(JP2-B) -> PWM_PIN2
- U6 pad 8: PWM_PIN2_O -> Net-(JP2-A)
Routing:
- net Net-(JP2-B): track 8.96 -> 0.00 mm
- net PWM_PIN2: track 56.9 -> 65.3 mm
- net +3V3: track 57.4 -> 65.1 mm, vias 20 -> 22
- net PWM_PIN2_O: track 29.0 -> 35.5 mm, vias 1 -> 2
- net Net-(JP2-A): track 0.00 -> 5.67 mm
- net SD_MOSI_GPIO_PIN4: track 69.7 -> 73.5 mm
- net SD_SCK_DAC_A8: track 62.7 -> 64.6 mm
- net SD_CS_PWM_26: track 65.4 -> 66.9 mm
- net SD_MISO_PWM_28: track 83.3 -> 84.5 mm
- net GND: track 158.5 -> 157.7 mm
Other:
- board size 110.2 x 53.8 mm -> 110.2 x 55.9 mm
- board text added: "0"
- board text added: "1"
- board text added: "10"
- board text added: "11"
- board text added: "12"
- board text added: "13"
- board text added: "14"
- board text added: "15"
- board text added: "16"
- board text added: "17"
- board text added: "18"
- board text added: "19"
- board text added: "2"
- board text added: "20"
- board text added: "21"
- board text added: "22"
- board text added: "23"
- board text added: "24"
- board text added: "25"
- board text added: "26"
- board text added: "27"
- board text added: "28"
- board text added: "29"
- board text added: "3"
- board text added: "3.3V"
- board text added: "30"
- board text added: "31"
- board text added: "32"
- board text added: "33"
- board text added: "34"
- board text added: "35"
- board text added: "36"
- board text added: "37"
- board text added: "38"
- board text added: "4"
- board text added: "5"
- board text added: "5V"
- board text added: "6"
- board text added: "7"
- board text added: "8"
- board text added: "9"
- board text added: "A0"
- board text added: "A1"
- board text added: "A2"
- board text added: "A3"
- board text added: "A4"
- board text added: "A5"
- board text added: "A6"
- board text added: "A7"
- board text added: "A8"
- board text added: "BOOT"
- board text added: "GND"
- board text added: "Hackboard"
- board text added: "IOREF"
- board text added: "RESET"
- board text added: "SCL"
- board text added: "SDA"
- board text added: "VDDA"
- board text added: "Vin"
- board text added: "adamturaj.com"
